Commit message: Changed Robot Model

File: roboticarm/urdf/robotic_arm.urdf (robot description, URDF)
Before this commit: robot roboticarm, 7 links, 6 joints
Links:
- removed link link_1
- removed link link_2
- removed link link_3
- removed link link_4
- removed link link_51
- removed link link_52
- added link arm_link_1, mass 0.19423597169735287715; collision mesh filename=package://roboticarm/meshes/arm_link_1.stl; visual mesh filename=package://roboticarm/meshes/arm_link_1.stl
- added link arm_link_2, mass 0.07194679150920589572; collision mesh filename=package://roboticarm/meshes/arm_link_2.stl; visual mesh filename=package://roboticarm/meshes/arm_link_2.stl
- added link arm_link_3, mass 0.04226949872412866932; collision mesh filename=package://roboticarm/meshes/arm_link_3.stl; visual mesh filename=package://roboticarm/meshes/arm_link_3.stl
- added link base_turner, mass 0.11175253124514644698; collision mesh filename=package://roboticarm/meshes/base_turner.stl; visual mesh filename=package://roboticarm/meshes/base_turner.stl
- added link gripper_link_1, mass 0.040925034173514361624; collision mesh filename=package://roboticarm/meshes/gripper_link_1.stl; visual mesh filename=package://roboticarm/meshes/gripper_link_1.stl
- added link gripper_link_2, mass 0.0062927985848676443875; collision mesh filename=package://roboticarm/meshes/gripper_link_2.stl; visual mesh filename=package://roboticarm/meshes/gripper_link_2.stl
- added link gripper_link_2_2, mass 0.0062927985848676443875; collision mesh filename=package://roboticarm/meshes/gripper_link_2.stl; visual mesh filename=package://roboticarm/meshes/gripper_link_2.stl
- added link gripper_link_3, mass 0.022194922914096641003; collision mesh filename=package://roboticarm/meshes/gripper_link_3.stl; visual mesh filename=package://roboticarm/meshes/gripper_link_3.stl
- added link gripper_link_4, mass 0.022194831460484187174; collision mesh filename=package://roboticarm/meshes/gripper_link_4.stl; visual mesh filename=package://roboticarm/meshes/gripper_link_4.stl
- added link world
- link base_link: mass 0.35184 -> 3; geometry collision mesh filename=package://roboticarm/meshes/base_link.stl; visual mesh filename=package://roboticarm/meshes/base_link.stl
Joints:
- removed joint joint_1
- removed joint joint_2
- removed joint joint_3
- removed joint joint_4
- removed joint joint_51
- removed joint joint_52
- added joint fixed: type fixed, parent world, child base_link
- added joint joint1: type revolute, parent base_link, child base_turner, origin xyz=7.3266230497424844212e-18 5.6144109730709618633e-19 0.020000000000000055927 rpy=-3.141592653589793116 -2.0000188391028945031e-17 -0.91339895386326697135, axis 0 0 1, limit lower=-3.14 upper=3.14 effort=100 velocity=1
- added joint joint2: type revolute, parent base_turner, child arm_link_1, origin xyz=1.7370716832809142268e-18 -0.020000000000000007355 -0.037500000000000005551 rpy=1.5707963267948956698 -1.5707963267948943376 0, axis 0 0 1, limit lower=-1.57 upper=1.57 effort=100 velocity=1
- added joint joint3: type revolute, parent arm_link_1, child arm_link_2, origin xyz=-0.13500000000000000888 3.0655396205876302604e-18 -0.040000000000000007772 rpy=1.566141830090408893e-15 2.5180549917200211291e-15 3.1415926535897868987, axis 0 0 1, limit lower=-1.7 upper=1.7 effort=100 velocity=1
- added joint joint4: type revolute, parent arm_link_2, child arm_link_3, origin xyz=0.075000000000000011102 2.1063240052122997717e-18 6.9388939039072283776e-18 rpy=-3.1415926535897926719 -2.4281616861104182506e-16 -3.1380330806969403135, axis 0 0 1, limit lower=-1.7 upper=1.7 effort=100 velocity=1
- added joint joint5: type revolute, parent arm_link_3, child gripper_link_1, origin xyz=-0.027500000000000024425 -8.2399365108898336985e-18 -0.020000000000000003886 rpy=3.141592653589793116 -1.5707963267948856778 0, axis 0 0 1, limit lower=-3.14 upper=3.14 effort=100 velocity=1
- added joint joint6: type revolute, parent gripper_link_1, child gripper_link_2, origin xyz=-0.014999999999999992506 0.0009999999999999993703 -0.019999999999999962252 rpy=1.570796326794896558 2.3228524371245603311e-14 -5.549460142490254044e-15, axis 0 0 1, limit lower=0 upper=0.2 effort=100 velocity=1
- added joint joint7: type revolute, parent gripper_link_1, child gripper_link_2_2, origin xyz=0.015000000000000004649 0.00099999999999999698505 -0.020000000000000017764 rpy=-1.570796326794896558 2.9211766417202967469e-14 3.1415926535897877869, axis 0 0 1, limit lower=-0.2 upper=0 effort=100 velocity=1
- added joint joint8: type revolute, parent gripper_link_2, child gripper_link_3, origin xyz=-0.040000000000000021649 -5.5511151231257827021e-17 3.1008182133085426813e-17 rpy=3.1415926535897926719 -4.8509407399613398583e-16 -1.570796326794896558, axis 0 0 1, limit lower=0 upper=0.2 effort=100 velocity=1
- added joint joint9: type revolute, parent gripper_link_2_2, child gripper_link_4, origin xyz=-0.040000000000000000833 -1.1102230246251565404e-16 1.8865117801247777152e-17 rpy=-3.1415926535897926719 1.2875113902521724409e-15 1.57079632679489678, axis 0 0 1, limit lower=-0.2 upper=0 effort=100 velocity=1

Commit message: Added final control claw code

File: roboticarm/urdf/robotic_arm.urdf (robot description, URDF)
Before this commit: robot roboticarm, 11 links, 10 joints
Joints:
- joint joint6: limit lower=0 upper=0.2 effort=100 velocity=1 -> lower=-1.57 upper=1.57 effort=100 velocity=1
- joint joint7: limit lower=-0.2 upper=0 effort=100 velocity=1 -> lower=-1.57 upper=1.57 effort=100 velocity=1
- joint joint8: limit lower=0 upper=0.2 effort=100 velocity=1 -> lower=-1.57 upper=1.57 effort=100 velocity=1
- joint joint9: limit lower=-0.2 upper=0 effort=100 velocity=1 -> lower=-1.57 upper=1.57 effort=100 velocity=1

Commit message: Formatted URDF

File: roboticarm/urdf/robotic_arm.urdf (robot description, URDF)
Before this commit: robot roboticarm, 11 links, 10 joints
Links:
- removed link world
- added link base_footprint
Joints:
- removed joint fixed
- added joint base_joint: type fixed, parent base_footprint, child base_link
