Commit message: Fixed no tf data error

File: roboticarm/urdf/robotic_arm.xacro (robot description, xacro)
@@ -1,4 +1,6 @@
 <?xml version="1.0" encoding="utf-8"?>
-<robot name="roboticarm">
+<robot name="roboticarm" xmlns:xacro="http://www.ros.org/wiki/xacro">
+<xacro:include filename="$(find roboticarm)/urdf/robotic_arm.trans" />
+<xacro:include filename="$(find roboticarm)/gazebo/robotic_arm_plugin.gazebo" />
 	<link name="base_link">
 		<visual>
@@ -23,7 +25,7 @@
 		</inertial>
 	</link>
-	<link name="base_footprint"/>
+	<link name="world"/>
   	<joint name="base_joint" type="fixed">
-    	<parent link="base_footprint"/>
+    	<parent link="world"/>
     	<child link="base_link"/>
   	</joint>
@@ -162,22 +164,22 @@
 	<link name="gripper_link_3">
 		<visual>
-		<origin xyz="0.030000000000000026645 -0.0030000000000000026645 -0.013500000000000003317" rpy="2.7895758333200453872e-17 -1.9176045572885558621e-19 5.9914972313653386157e-19" />
-		<geometry>
-		<mesh filename="package://roboticarm/meshes/gripper_link_3.stl"/>
-		</geometry>
-		<material name="gripper_link_3_material">
-		<color rgba="0 0 0 1.0"/>
-		</material>
-		</visual>
-		<collision>
-		<origin xyz="0.030000000000000026645 -0.0030000000000000026645 -0.013500000000000003317" rpy="2.7895758333200453872e-17 -1.9176045572885558621e-19 5.9914972313653386157e-19" />
-		<geometry>
-		<mesh filename="package://roboticarm/meshes/gripper_link_3.stl"/>
-		</geometry>
-		</collision>
-		<inertial>
-		<origin xyz="0.047860279909926396746 -0.001816675545418268943 -0.0023582232389542500534" rpy="0 0 0"/>
-		<mass value="0.022194922914096641003" />
-		<inertia ixx="1.4659648868937333891e-06" ixy="1.0083147605711552851e-06"  ixz="-1.0394543711540078819e-06" iyy="1.4282656004211426759e-05" iyz="7.2086988985399456882e-08" izz="1.352743129292048836e-05" />
+			<origin xyz="0.030000000000000026645 -0.0030000000000000026645 -0.013500000000000003317" rpy="2.7895758333200453872e-17 -1.9176045572885558621e-19 5.9914972313653386157e-19" />
+			<geometry>
+				<mesh filename="package://roboticarm/meshes/gripper_link_3.stl"/>
+			</geometry>
+			<material name="gripper_link_3_material">
+				<color rgba="0 0 0 1.0"/>
+			</material>
+		</visual>
+		<collision>
+			<origin xyz="0.030000000000000026645 -0.0030000000000000026645 -0.013500000000000003317" rpy="2.7895758333200453872e-17 -1.9176045572885558621e-19 5.9914972313653386157e-19" />
+			<geometry>
+				<mesh filename="package://roboticarm/meshes/gripper_link_3.stl"/>
+			</geometry>
+		</collision>
+		<inertial>
+			<origin xyz="0.047860279909926396746 -0.001816675545418268943 -0.0023582232389542500534" rpy="0 0 0"/>
+			<mass value="0.022194922914096641003" />
+			<inertia ixx="1.4659648868937333891e-06" ixy="1.0083147605711552851e-06"  ixz="-1.0394543711540078819e-06" iyy="1.4282656004211426759e-05" iyz="7.2086988985399456882e-08" izz="1.352743129292048836e-05" />
 		</inertial>
 	</link>
@@ -289,90 +291,3 @@
 		<limit lower="-3.14" upper="3.14" effort="100" velocity="1" />
 	</joint>
-	<!-- gazebo related stuffs -->
-	<gazebo>
-		<plugin name="gazebo_ros_control" filename="libgazebo_ros_control.so">
-			<robotNamespace>/roboticarm</robotNamespace>
-		</plugin>
-	</gazebo>
-	<transmission name="trans_1">
-		<type>transmission_interface/SimpleTransmission</type>
-		<joint name="joint1">
-			<hardwareInterface>hardware_interface/EffortJointInterface</hardwareInterface>
-		</joint>
-		<actuator name="motor_1">
-			<mechanicalReduction>10</mechanicalReduction>
-		</actuator>
-	</transmission>
-	<transmission name="trans_2">
-		<type>transmission_interface/SimpleTransmission</type>
-		<joint name="joint2">
-			<hardwareInterface>hardware_interface/EffortJointInterface</hardwareInterface>
-		</joint>
-		<actuator name="motor_2">
-			<mechanicalReduction>10</mechanicalReduction>
-		</actuator>
-	</transmission>
-	<transmission name="trans_3">
-		<type>transmission_interface/SimpleTransmission</type>
-		<joint name="joint3">
-			<hardwareInterface>hardware_interface/EffortJointInterface</hardwareInterface>
-		</joint>
-		<actuator name="motor_3">
-			<mechanicalReduction>10</mechanicalReduction>
-		</actuator>
-	</transmission>
-	<transmission name="trans_4">
-		<type>transmission_interface/SimpleTransmission</type>
-		<joint name="joint4">
-			<hardwareInterface>hardware_interface/EffortJointInterface</hardwareInterface>
-		</joint>
-		<actuator name="motor_4">
-			<mechanicalReduction>10</mechanicalReduction>
-		</actuator>
-	</transmission>
-	<transmission name="trans_5">
-		<type>transmission_interface/SimpleTransmission</type>
-		<joint name="joint5">
-			<hardwareInterface>hardware_interface/EffortJointInterface</hardwareInterface>
-		</joint>
-		<actuator name="motor_5">
-			<mechanicalReduction>10</mechanicalReduction>
-		</actuator>
-	</transmission>
-	<transmission name="trans_6">
-		<type>transmission_interface/SimpleTransmission</type>
-		<joint name="joint6">
-			<hardwareInterface>hardware_interface/EffortJointInterface</hardwareInterface>
-		</joint>
-		<actuator name="motor_6">
-			<mechanicalReduction>10</mechanicalReduction>
-		</actuator>
-	</transmission>
-	<transmission name="trans_7">
-		<type>transmission_interface/SimpleTransmission</type>
-		<joint name="joint7">
-			<hardwareInterface>hardware_interface/EffortJointInterface</hardwareInterface>
-		</joint>
-		<actuator name="motor_7">
-			<mechanicalReduction>10</mechanicalReduction>
-		</actuator>
-	</transmission>
-	<transmission name="trans_8">
-		<type>transmission_interface/SimpleTransmission</type>
-		<joint name="joint8">
-			<hardwareInterface>hardware_interface/EffortJointInterface</hardwareInterface>
-		</joint>
-		<actuator name="motor_8">
-			<mechanicalReduction>10</mechanicalReduction>
-		</actuator>
-	</transmission>
-	<transmission name="trans_9">
-		<type>transmission_interface/SimpleTransmission</type>
-		<joint name="joint9">
-			<hardwareInterface>hardware_interface/EffortJointInterface</hardwareInterface>
-		</joint>
-		<actuator name="motor_9">
-			<mechanicalReduction>10</mechanicalReduction>
-		</actuator>
-	</transmission>
 </robot>

Commit message: Added materials to simulation model

File: roboticarm/urdf/robotic_arm.xacro (robot description, xacro)
@@ -3,4 +3,5 @@
 <xacro:include filename="$(find roboticarm)/urdf/robotic_arm.trans" />
 <xacro:include filename="$(find roboticarm)/gazebo/robotic_arm_plugin.gazebo" />
+<xacro:include filename="$(find roboticarm)/gazebo/robotic_arm_material.gazebo" />
 	<link name="base_link">
 		<visual>
@@ -198,5 +199,5 @@
 		<limit lower="-1.57" upper="1.57" effort="100" velocity="1" />
 	</joint>
-	<link name="gripper_link_2_2">
+	<link name="gripper_link_4">
 		<visual>
 			<origin xyz="-0.020000000000000003886 0 -0.01249999999999999549" rpy="-1.8231828477160622874e-19 4.5024695016245069465e-17 -3.467885654086683229e-20" />
@@ -220,5 +221,5 @@
 		</inertial>
 	</link>
-	<link name="gripper_link_4">
+	<link name="gripper_link_5">
 		<visual>
 			<origin xyz="0.030000000000000026645 0.0030000000000000026645 -0.00099999999999999915345" rpy="-3.141592653589793116 -3.5474759767231887989e-19 1.5061988724684013876e-19" />
@@ -226,5 +227,5 @@
 				<mesh filename="package://roboticarm/meshes/gripper_link_4.stl"/>
 			</geometry>
-			<material name="gripper_link_4_material">
+			<material name="gripper_link_5_material">
 				<color rgba="0 0 0 1.0"/>
 			</material>
@@ -244,6 +245,6 @@
 	<joint name="joint9" type="revolute">
 		<origin xyz="-0.040000000000000000833 -1.1102230246251565404e-16 1.8865117801247777152e-17" rpy="-3.1415926535897926719 1.2875113902521724409e-15 1.57079632679489678" />
-		<parent link="gripper_link_2_2" />
-		<child link="gripper_link_4" />
+		<parent link="gripper_link_4" />
+		<child link="gripper_link_5" />
 		<axis xyz="0 0 1"/>
 		<limit lower="-1.57" upper="1.57" effort="100" velocity="1" />
@@ -252,5 +253,5 @@
 		<origin xyz="0.015000000000000004649 0.00099999999999999698505 -0.020000000000000017764" rpy="-1.570796326794896558 2.9211766417202967469e-14 3.1415926535897877869" />
 		<parent link="gripper_link_1" />
-		<child link="gripper_link_2_2" />
+		<child link="gripper_link_4" />
 		<axis xyz="0 0 1"/>
 		<limit lower="-1.57" upper="1.57" effort="100" velocity="1" />
